File: avrsheild/avrsheild.kicad_sch (KiCad schematic)
At the start: 21 parts, among them J1 USB-C, J2 portD, J3 portC, J4 portB, SW1 SW_Push, U1 ATmega328P-P, U2 CH340C, Y1 Crystal

Commit message: PCB layout is done
Parts:
- added J5: Power_pin, Connector_PinHeader_2.54mm:PinHeader_1x03_P2.54mm_Horizontal, symbol Connector:Conn_01x03_Pin
Connections:
- net +5V: now also J5.3 (Pin_3)
- net GND: now also J5.2 (Pin_2)
- net at U2.5 (UD+): now also J1.3 (Pin_3); no longer J1.2 (Pin_2)
- net at U2.6 (UD-): now also J1.2 (Pin_2); no longer J1.3 (Pin_3)
- net at C4.2, R1.1, SW1.1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: now also J5.1 (Pin_1)
- net at D2.2 (A), J4.6 (Pin_6), U1.19 (PB5): no longer C2.1, U1.9 (XTAL1/PB6), Y1.1
- new net: C2.1, U1.9 (XTAL1/PB6), Y1.1
